File: Hardware/ISP_Pogo_Board.sch (EAGLE design)
At the start: 12 parts, among them J2 AVR_SPI_PRG_6NS

Commit message: Changed for v10: Made planes not overlap vscore region Increased annular ring on pogo pin pads
Other:
- note added: "10"
- note removed: "02"
Changed lines of the file:
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@@
 <plain>
 <text x="172.72" y="7.62" size="5.08" layer="94">M.HORD</text>
-<text x="239.014" y="6.604" size="3.81" layer="94">02</text>
+<text x="239.014" y="6.604" size="3.81" layer="94">10</text>
 </plain>
 <instances>
@@
 <segment>
 <pinref part="J1" gate="G$1" pin="1"/>
-<wire x1="119.38" y1="132.08" x2="116.84" y2="132.08" width="0.1524" layer="91"/>
+<wire x1="121.92" y1="132.08" x2="116.84" y2="132.08" width="0.1524" layer="91"/>
 <wire x1="116.84" y1="132.08" x2="116.84" y2="109.22" width="0.1524" layer="91"/>
 <pinref part="J2" gate="G$1" pin="1"/>
@@
 <segment>
 <pinref part="J1" gate="G$1" pin="3"/>
-<wire x1="119.38" y1="129.54" x2="114.3" y2="129.54" width="0.1524" layer="91"/>
+<wire x1="121.92" y1="129.54" x2="114.3" y2="129.54" width="0.1524" layer="91"/>
 <wire x1="114.3" y1="129.54" x2="114.3" y2="106.68" width="0.1524" layer="91"/>
 <pinref part="J2" gate="G$1" pin="3"/>
@@
 <segment>
 <pinref part="J1" gate="G$1" pin="5"/>
-<wire x1="119.38" y1="127" x2="111.76" y2="127" width="0.1524" layer="91"/>
+<wire x1="121.92" y1="127" x2="111.76" y2="127" width="0.1524" layer="91"/>
 <wire x1="111.76" y1="127" x2="111.76" y2="104.14" width="0.1524" layer="91"/>
 <pinref part="J2" gate="G$1" pin="5"/>
@@
 <segment>
 <pinref part="J1" gate="G$1" pin="2"/>
-<wire x1="139.7" y1="132.08" x2="144.78" y2="132.08" width="0.1524" layer="91"/>
+<wire x1="137.16" y1="132.08" x2="144.78" y2="132.08" width="0.1524" layer="91"/>
 <wire x1="144.78" y1="132.08" x2="144.78" y2="121.92" width="0.1524" layer="91"/>
 <pinref part="J2" gate="G$1" pin="2"/>
@@
 <segment>
 <pinref part="J1" gate="G$1" pin="4"/>
-<wire x1="139.7" y1="129.54" x2="147.32" y2="129.54" width="0.1524" layer="91"/>
+<wire x1="137.16" y1="129.54" x2="147.32" y2="129.54" width="0.1524" layer="91"/>
 <pinref part="J2" gate="G$1" pin="4"/>
 <wire x1="147.32" y1="129.54" x2="147.32" y2="119.38" width="0.1524" layer="91"/>
@@
 <segment>
 <pinref part="J1" gate="G$1" pin="6"/>
-<wire x1="139.7" y1="127" x2="149.86" y2="127" width="0.1524" layer="91"/>
+<wire x1="137.16" y1="127" x2="149.86" y2="127" width="0.1524" layer="91"/>
 <pinref part="J2" gate="G$1" pin="6"/>
 <wire x1="149.86" y1="127" x2="149.86" y2="116.84" width="0.1524" layer="91"/>
@@
 <pinref part="J4" gate="G$1" pin="+"/>
 <pinref part="J3" gate="G$1" pin="2"/>
-<wire x1="149.86" y1="78.74" x2="142.24" y2="78.74" width="0.1524" layer="91"/>
+<wire x1="149.86" y1="78.74" x2="139.7" y2="78.74" width="0.1524" layer="91"/>
 </segment>
 </net>
@@
 <wire x1="144.78" y1="76.2" x2="144.78" y2="73.66" width="0.1524" layer="91"/>
 <pinref part="J3" gate="G$1" pin="6"/>
-<wire x1="144.78" y1="73.66" x2="142.24" y2="73.66" width="0.1524" layer="91"/>
+<wire x1="144.78" y1="73.66" x2="139.7" y2="73.66" width="0.1524" layer="91"/>
 </segment>
 </net>
